Commit message: 0625 2208

File: IsaacGymEnvs/assets/urdf/PongBot_R_V1/urdf/PongBot_R_V1_(train).urdf (robot description, URDF)
Before this commit: robot PongBot_R_V1.0, 17 links, 16 joints
Joints:
- joint FL_HP_JOINT: limit lower=-0.366519 upper=1.5708 effort=200 velocity=13 -> lower=-0.366519 upper=1.5708 effort=80 velocity=13
- joint FL_HR_JOINT: limit lower=-0.349066 upper=0.349066 effort=200 velocity=13 -> lower=-0.349066 upper=0.349066 effort=80 velocity=13
- joint FL_KN_JOINT: limit lower=-2.58309 upper=-0.488692 effort=200 velocity=13 -> lower=-2.58309 upper=-0.488692 effort=80 velocity=13
- joint FR_HP_JOINT: limit lower=-0.366519 upper=1.5708 effort=200 velocity=13 -> lower=-0.366519 upper=1.5708 effort=80 velocity=13
- joint FR_HR_JOINT: limit lower=-0.349066 upper=0.349066 effort=200 velocity=13 -> lower=-0.349066 upper=0.349066 effort=80 velocity=13
- joint FR_KN_JOINT: limit lower=-2.58309 upper=-0.488692 effort=200 velocity=13 -> lower=-2.58309 upper=-0.488692 effort=80 velocity=13
- joint RL_HP_JOINT: limit lower=-0.366519 upper=1.5708 effort=200 velocity=13 -> lower=-0.366519 upper=1.5708 effort=80 velocity=13
- joint RL_HR_JOINT: limit lower=-0.349066 upper=0.349066 effort=200 velocity=13 -> lower=-0.349066 upper=0.349066 effort=80 velocity=13
- joint RL_KN_JOINT: limit lower=-2.58309 upper=-0.488692 effort=200 velocity=13 -> lower=-2.58309 upper=-0.488692 effort=80 velocity=13
- joint RR_HP_JOINT: limit lower=-0.366519 upper=1.5708 effort=200 velocity=13 -> lower=-0.366519 upper=1.5708 effort=80 velocity=13
- joint RR_HR_JOINT: limit lower=-0.349066 upper=0.349066 effort=200 velocity=13 -> lower=-0.349066 upper=0.349066 effort=80 velocity=13
- joint RR_KN_JOINT: limit lower=-2.58309 upper=-0.488692 effort=200 velocity=13 -> lower=-2.58309 upper=-0.488692 effort=80 velocity=13
